Commit message: IMU support to control End Effector orientation, offset accounted for according to IMU placement

File: src/kinova_description/urdf/gen3_7dof_novision.xacro (robot description, xacro)
@@ -50,5 +50,5 @@
     <child link="shoulder_link" />
     <axis xyz="0 0 1" />
-    <limit effort="39" velocity="1.3963" />
+    <limit effort="39" velocity="1.0" />
   </joint>
   <link name="half_arm_1_link">
@@ -79,5 +79,5 @@
     <child link="half_arm_1_link" />
     <axis xyz="0 0 1" />
-    <limit lower="-2.24" upper="2.24" effort="39" velocity="1.3963" />
+    <limit lower="-2.24" upper="2.24" effort="39" velocity="1.0" />
   </joint>
   <link name="half_arm_2_link">
@@ -108,5 +108,5 @@
     <child link="half_arm_2_link" />
     <axis xyz="0 0 1" />
-    <limit effort="39" velocity="1.3963" />
+    <limit effort="39" velocity="1.0" />
   </joint>
   <link name="forearm_link">
@@ -137,5 +137,5 @@
     <child link="forearm_link" />
     <axis xyz="0 0 1" />
-    <limit lower="-2.57" upper="2.57" effort="39" velocity="1.3963" />
+    <limit lower="-2.57" upper="2.57" effort="39" velocity="1.0" />
   </joint>
   <link name="spherical_wrist_1_link">
@@ -166,5 +166,5 @@
     <child link="spherical_wrist_1_link" />
     <axis xyz="0 0 1" />
-    <limit effort="9" velocity="1.2218" />
+    <limit effort="9" velocity="1.0" />
   </joint>
   <link name="spherical_wrist_2_link">
@@ -195,5 +195,5 @@
     <child link="spherical_wrist_2_link" />
     <axis xyz="0 0 1" />
-    <limit lower="-2.09" upper="2.09" effort="9" velocity="1.2218" />
+    <limit lower="-2.09" upper="2.09" effort="9" velocity="1.0" />
   </joint>
   <link name="bracelet_link">
@@ -224,5 +224,5 @@
     <child link="bracelet_link" />
     <axis xyz="0 0 1" />
-    <limit effort="9" velocity="1.2218" />
+    <limit effort="9" velocity="1.0" />
   </joint>
   <link name="end_effector_link">

Commit message: added logging of data

File: src/kinova_description/urdf/gen3_7dof_novision.xacro (robot description, xacro)
@@ -50,5 +50,5 @@
     <child link="shoulder_link" />
     <axis xyz="0 0 1" />
-    <limit effort="39" velocity="1.0" />
+    <limit effort="39" velocity="1.3" />
   </joint>
   <link name="half_arm_1_link">
@@ -79,5 +79,5 @@
     <child link="half_arm_1_link" />
     <axis xyz="0 0 1" />
-    <limit lower="-2.24" upper="2.24" effort="39" velocity="1.0" />
+    <limit lower="-2.24" upper="2.24" effort="39" velocity="1.3" />
   </joint>
   <link name="half_arm_2_link">
@@ -108,5 +108,5 @@
     <child link="half_arm_2_link" />
     <axis xyz="0 0 1" />
-    <limit effort="39" velocity="1.0" />
+    <limit effort="39" velocity="1.3" />
   </joint>
   <link name="forearm_link">
@@ -137,5 +137,5 @@
     <child link="forearm_link" />
     <axis xyz="0 0 1" />
-    <limit lower="-2.57" upper="2.57" effort="39" velocity="1.0" />
+    <limit lower="-2.57" upper="2.57" effort="39" velocity="1.3" />
   </joint>
   <link name="spherical_wrist_1_link">
@@ -166,5 +166,5 @@
     <child link="spherical_wrist_1_link" />
     <axis xyz="0 0 1" />
-    <limit effort="9" velocity="1.0" />
+    <limit effort="9" velocity="1.3" />
   </joint>
   <link name="spherical_wrist_2_link">
@@ -195,5 +195,5 @@
     <child link="spherical_wrist_2_link" />
     <axis xyz="0 0 1" />
-    <limit lower="-2.09" upper="2.09" effort="9" velocity="1.0" />
+    <limit lower="-2.09" upper="2.09" effort="9" velocity="1.3" />
   </joint>
   <link name="bracelet_link">
@@ -224,5 +224,5 @@
     <child link="bracelet_link" />
     <axis xyz="0 0 1" />
-    <limit effort="9" velocity="1.0" />
+    <limit effort="9" velocity="1.3" />
   </joint>
   <link name="end_effector_link">

Commit message: Arduino Code added

File: src/kinova_description/urdf/gen3_7dof_novision.xacro (robot description, xacro)
@@ -50,5 +50,5 @@
     <child link="shoulder_link" />
     <axis xyz="0 0 1" />
-    <limit effort="39" velocity="1.3" />
+    <limit effort="39" velocity="2.0" />
   </joint>
   <link name="half_arm_1_link">
@@ -79,5 +79,5 @@
     <child link="half_arm_1_link" />
     <axis xyz="0 0 1" />
-    <limit lower="-2.24" upper="2.24" effort="39" velocity="1.3" />
+    <limit lower="-2.24" upper="2.24" effort="39" velocity="2.0" />
   </joint>
   <link name="half_arm_2_link">
@@ -108,5 +108,5 @@
     <child link="half_arm_2_link" />
     <axis xyz="0 0 1" />
-    <limit effort="39" velocity="1.3" />
+    <limit effort="39" velocity="2.0" />
   </joint>
   <link name="forearm_link">
@@ -137,5 +137,5 @@
     <child link="forearm_link" />
     <axis xyz="0 0 1" />
-    <limit lower="-2.57" upper="2.57" effort="39" velocity="1.3" />
+    <limit lower="-2.57" upper="2.57" effort="39" velocity="2.0" />
   </joint>
   <link name="spherical_wrist_1_link">
@@ -166,5 +166,5 @@
     <child link="spherical_wrist_1_link" />
     <axis xyz="0 0 1" />
-    <limit effort="9" velocity="1.3" />
+    <limit effort="9" velocity="2.0" />
   </joint>
   <link name="spherical_wrist_2_link">
@@ -195,5 +195,5 @@
     <child link="spherical_wrist_2_link" />
     <axis xyz="0 0 1" />
-    <limit lower="-2.09" upper="2.09" effort="9" velocity="1.3" />
+    <limit lower="-2.09" upper="2.09" effort="9" velocity="2.0" />
   </joint>
   <link name="bracelet_link">
@@ -224,5 +224,5 @@
     <child link="bracelet_link" />
     <axis xyz="0 0 1" />
-    <limit effort="9" velocity="1.3" />
+    <limit effort="9" velocity="2.0" />
   </joint>
   <link name="end_effector_link">
